File: PCB/SpringReverbRev2.1_combined.sch (EAGLE design)
At the start: 85 parts, among them IC102 TL074, IC103 TL074, J1 MA08-1, J2 MA08-1, U1 TL072_, U2 TL072_, U7 NE5532

Commit message: Fixes #18
Connections:
- removed net N$14: JP101.1
- net S+: now also JP101.1
Changed lines of the file:
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@@
 <segment>
 <wire x1="66.04" y1="251.46" x2="66.04" y2="248.92" width="0.1524" layer="91"/>
-<wire x1="66.04" y1="248.92" x2="66.04" y2="241.3" width="0.1524" layer="91"/>
+<wire x1="66.04" y1="248.92" x2="66.04" y2="246.38" width="0.1524" layer="91"/>
+<wire x1="66.04" y1="246.38" x2="66.04" y2="241.3" width="0.1524" layer="91"/>
 <wire x1="27.94" y1="259.08" x2="20.32" y2="259.08" width="0.1524" layer="91"/>
 <wire x1="20.32" y1="259.08" x2="20.32" y2="241.3" width="0.1524" layer="91"/>
@@
 <pinref part="TO_TANK" gate="G$1" pin="SLEEVE"/>
 <junction x="66.04" y="248.92"/>
+<pinref part="JP101" gate="G$1" pin="1"/>
+<wire x1="78.74" y1="259.08" x2="78.74" y2="246.38" width="0.1524" layer="91"/>
+<wire x1="78.74" y1="246.38" x2="66.04" y2="246.38" width="0.1524" layer="91"/>
+<junction x="66.04" y="246.38"/>
 </segment>
 </net>
@@
 </segment>
 </net>
-<net name="N$14" class="0">
-<segment>
-<pinref part="JP101" gate="G$1" pin="1"/>
-<wire x1="78.74" y1="259.08" x2="78.74" y2="246.38" width="0.1524" layer="91"/>
-</segment>
-</net>
